File: pcb/loraPowerUp.kicad_pcb (KiCad board)
At the start: 2 copper layers, 27 x 28.5 mm, 10 parts, among them P1_L1 IN_LEFT, P1_R1 IN_RIGHT, P2_L1 DORGI_L, P2_R1 DORGI_R, P3 LORA, Q1 NPN, Q2 P-FET

Commit message: Fixing VCC
Parts:
- Q1: value NPN -> Q_NPN_BCE
- Q2: value P-FET -> IRF9540N
Connections:
- P1_R1 pad 1: LoRaVCC -> VCC
- Q2 pad 2: LoRaVCC -> VCC
- R3 pad 1: LoRaVCC -> VCC
Routing:
- net VCC: track 0.00 -> 31.1 mm
- net GND: track 67.0 -> 55.4 mm, vias 1 -> 0
- net LoRaVCC: track 55.2 -> 44.5 mm
- net Net-(Q1-Pad2): track 11.5 -> 12.8 mm
- removed copper zone on B.Cu, net GND
- removed copper zone on F.Cu, net GND
